Commit message: modify config files

File: src/cartographer_ros/cartographer_ros/urdf/test_2d.urdf (robot description, URDF)
Before this commit: robot cartographer_backpack_2d, 4 links, 3 joints
Links:
- removed link lidar_frame
- removed link vertical_laser_link
- added link horizontal_laser_link; visual cylinder length=0.05 radius=0.03
Joints:
- removed joint lidar_frame_joint
- removed joint vertical_laser_link_joint
- added joint horizontal_laser_link_joint: type fixed, parent base_link, child horizontal_laser_link, origin xyz=0 0 0
